File: electronics/distro/distro.kicad_pcb (KiCad board)
At the start: 2 copper layers, 24 parts

Commit message: distro work
Parts:
- removed BH1, BH2: 4mm, MountingHole:MountingHole_4.3mm_M4
- removed H5, H6, H7, H8: M3, MountingHole:MountingHole_3.2mm_M3
- moved TG1 194.0 mm to (71.2, 46.8)
- moved TM2 179.3 mm to (100.3, 45.5), turned to 180 degrees
- moved H2 165.0 mm to (62.5, 43.5), turned to 90 degrees
- moved H1 160.6 mm to (62.5, 78.5), turned to 90 degrees
- moved TG2 121.5 mm to (147.4, 72.2)
- moved FW1 118.8 mm to (74.8, 55.8)
- moved TM1 107.3 mm to (157.5, 74.8), turned to 180 degrees
- moved FW2 97.7 mm to (100.2, 68.5)
- moved BT1 93.7 mm to (165.9, 25.5)
- moved BR1 83.0 mm to (109.0, 55.0)
- moved D1 76.2 mm to (153.8, 49.5), turned to 180 degrees
- moved JFC1 73.5 mm to (178.0, 63.2)
- moved H4 69.8 mm to (182.5, 43.5), turned to 90 degrees
- moved JPY2 65.4 mm to (82.5, 77.0), turned to 90 degrees
- moved H3 57.9 mm to (182.5, 78.5), turned to 90 degrees
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Other:
- board outline added: 127 x 42 mm
