File: electronics/distro/distro.kicad_sch (KiCad schematic)
At the start: 24 parts

Commit message: distro work
Parts:
- removed BH1, BH2: 4mm, MountingHole:MountingHole_4.3mm_M4, symbol Mechanical:MountingHole
- removed H5, H6, H7, H8: M3, MountingHole:MountingHole_3.2mm_M3, symbol Mechanical:MountingHole
Other:
- moved on the sheet: H3, H4
